Commit message: Add files via upload

File: urdf_tutorial/urdf/my_robot.urdf (robot description, URDF)
Before this commit: robot test_robot, 5 links, 4 joints
Joints:
- joint joint1: origin xyz=0 0 0.75 rpy=-1.57 0 0 -> xyz=0 0 0.75 rpy=-1.57 0 1.57
- joint joint2: axis 0 0 1 -> 0 1 0; limit lower=-1 upper=1 effort=10.0 velocity=0.5 -> lower=0 upper=1 effort=10.0 velocity=0.5; origin xyz=0 -0.07 0  rpy=-1.57 0 -1.57 -> xyz=0 -0.07 0  rpy=1.57 3.14 1.57
- joint joint3: axis 1 0 0 -> 0 1 0; limit lower=-1 upper=1 effort=10.0 velocity=0.5 -> lower=0 upper=1 effort=10.0 velocity=0.5; origin xyz=0 -1 0 rpy=1.57 0 -1.57 -> xyz=0 0 1 rpy=1.57 3.14 -1.57
